File: qs75.kicad_pcb (KiCad board)
At the start: 2 copper layers, 285 x 95.1 mm, 286 parts, among them J1 SWD, J2 SPI, J3 UART, J4 USB2.0, J5 PB14, SW1 SW_Push, SW10 1u, SW11 1u, SW12 1u, SW13 1u, SW14 1u, SW15 1u, SW16 1u, SW17 1u, SW18 1u, SW19 1u, SW2 1u, SW20 1u, SW21 1u, SW22 1u, SW23 1u, SW24 1u, SW25 1u, SW26 1u, SW27 1u, SW28 1u, SW29 1u, SW3 1u, SW30 1u, SW31 1u, SW32 1u, SW33 1u, SW34 1u, SW35 1u, SW36 1u, SW37 1u, SW38 1u, SW39 1u, SW4 1u, SW40 1u, SW41 1u, SW42 1u, SW43 1u, SW44 1u, SW45 1u, SW46 1u, SW47 1u, SW48 1u, SW49 1u, SW5 1u, SW50 1u, SW51 1u, SW52 1u, SW53 1u, SW54 1u, SW55 1u, SW56 1u, SW57 1u, SW58 1u, SW59 1u, SW6 1u, SW60 1u, SW61 1u, SW62 1u, SW63 1u, SW64 1u, SW65 1u, SW66 1u, SW67 1u, SW68 1u, SW69 1u, SW7 1u, SW70 1u, SW71 1u, SW72 1u, SW73 1u, SW74 1u, SW75 1u, SW76 1u, SW8 1u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

Commit message: Change layout
Parts:
- removed the HOLE at (290.3, 76.4)
- removed the HOLE at (8.16, 76.4)
- removed JP2, JP5: Jumper_3_Open, Jumper:SolderJumper-3_P1.3mm_Open_RoundedPad1.0x1.5mm_NumberLabels
- removed LS2: Speaker, locallib:Buzzer_CUI_CPT-9019S-SMT
- added HOLE: VAL**, hole:PKRHSL, F.Cu at (290.3, 76.4)
- added HOLE: VAL**, hole:PKRHSL, F.Cu at (8.17, 76.4)
- added SW77: SW_Push, Button_Switch_SMD:SW_Push_SPST_NO_Alps_SKRK, B.Cu at (29.8, 64.7)
- U1, U2: footprint locallib:qfn40 -> locallib:qfn-40-5x5mm
- moved D32 1.34 mm to (27.9, 68.6)
- moved SW22 0.76 mm to (111.0, 48.2)
- moved U2 0.50 mm to (177.7, 41.6)
- moved U1 0.31 mm to (120.2, 41.3)
- moved C5 0.23 mm to (33.5, 76.3)
- moved C2 0.22 mm to (36.5, 76.3)
- moved R3 0.20 mm to (35.0, 76.3)
Connections:
- LS1 pad 2: Net-(JP2-Pad2) -> PA5
- U1 pad 27: (no net) -> aCS11
- U1 pad 28: (no net) -> aCS12
- U1 pad 37: (no net) -> Net-(U1-Pad37)
- U2 pad 27: (no net) -> bCS11
- U2 pad 28: (no net) -> bCS12
- U2 pad 37: (no net) -> Net-(U2-Pad37)
- U5 pad 4: (no net) -> Net-(U5-Pad4)
- USB1 pad 3: (no net) -> Net-(USB1-Pad3)
- USB1 pad 9: (no net) -> Net-(USB1-Pad9)
Routing:
- net Net-(JP5-Pad2): track 231.3 -> 0.00 mm, vias 2 -> 0
- net PA5: track 284.4 -> 62.1 mm, vias 2 -> 0
- net bSW3: track 263.7 -> 314.2 mm, vias 2 -> 6
- net aSW6: track 389.8 -> 419.7 mm, vias 8 -> 13
- net +5V: track 321.2 -> 295.2 mm
- net Net-(JP2-Pad2): track 23.7 -> 0.00 mm
- net bCS2: track 70.8 -> 90.4 mm
- net +3V3: track 535.1 -> 550.7 mm
- net Net-(R3-Pad1): track 14.1 -> 27.7 mm, vias 2 -> 3
- net bCS1: track 76.7 -> 89.8 mm
- net bCS4: track 144.8 -> 156.6 mm
- net bCS5: track 143.2 -> 155.0 mm
- net aCS8: track 107.9 -> 119.6 mm
- net bCS8: track 140.2 -> 151.0 mm
- net aCS9: track 185.2 -> 195.3 mm
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Other:
- outline, holes or cut-outs redrawn
- net class Default: clearance 0.2 -> 0.15
- net class Power: clearance 0.2 -> 0.15
- rule trace_clearance: 0.2 -> 0.15

Commit message: Reroute tracks
Parts:
- moved R16 0.38 mm to (24.5, 41.7)
- moved D17 0.07 mm to (27.9, 48.2)
Routing:
- net +5V: track 295.2 -> 426.9 mm, vias 9 -> 11
- net +3V3: track 550.7 -> 668.7 mm
- net GND: track 1109.1 -> 1042.4 mm, vias 400 -> 445
- net VCC: track 42.6 -> 59.2 mm
- net ROW3: track 352.8 -> 336.4 mm
- net aSW12: track 300.5 -> 292.5 mm
- net bSW10: track 150.8 -> 157.4 mm
- net aCS9: track 195.3 -> 200.6 mm
- net aSW4: track 369.9 -> 364.7 mm
- net aSW5: track 347.2 -> 351.3 mm
- net bSW6: track 283.1 -> 286.9 mm
- net aSW1: track 312.9 -> 316.6 mm
- net bSW5: track 337.4 -> 334.4 mm
- net aCS8: track 119.6 -> 122.4 mm
- net aSW10: track 280.7 -> 283.5 mm
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Other:
- net class Default: clearance 0.15 -> 0.2
- net class Power: clearance 0.15 -> 0.2; trace_width 0.381 -> 0.508
- rule trace_clearance: 0.15 -> 0.2

Commit message: Add tracks
Parts:
- turned D1 to 90 degrees
- turned D10 to 90 degrees
- turned D11 to 90 degrees
- turned D12 to 90 degrees
- turned D13 to 90 degrees
- turned D15 to 90 degrees
- turned D16 to 90 degrees
- turned D17 to 90 degrees
- turned D18 to 90 degrees
- turned D19 to 90 degrees
- turned D2 to 0 degrees
- turned D20 to 90 degrees
- turned D21 to 90 degrees
- turned D22 to 90 degrees
- turned D23 to 90 degrees
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Connections:
- D1 pad 1: ROW0 -> Net-(D1-Pad1)
- D1 pad 2: Net-(D1-Pad2) -> ROW0
- D10 pad 1: ROW0 -> Net-(D10-Pad1)
- D10 pad 2: Net-(D10-Pad2) -> ROW0
- D11 pad 1: ROW0 -> Net-(D11-Pad1)
- D11 pad 2: Net-(D11-Pad2) -> ROW0
- D12 pad 1: ROW0 -> Net-(D12-Pad1)
- D12 pad 2: Net-(D12-Pad2) -> ROW0
- D13 pad 1: ROW0 -> Net-(D13-Pad1)
- D13 pad 2: Net-(D13-Pad2) -> ROW0
- D15 pad 1: ROW0 -> Net-(D15-Pad1)
- D15 pad 2: Net-(D15-Pad2) -> ROW0
- D16 pad 1: ROW1 -> Net-(D16-Pad1)
- D16 pad 2: Net-(D16-Pad2) -> ROW1
- D17 pad 1: ROW1 -> Net-(D17-Pad1)
- D17 pad 2: Net-(D17-Pad2) -> ROW1
- D18 pad 1: ROW1 -> Net-(D18-Pad1)
- D18 pad 2: Net-(D18-Pad2) -> ROW1
- D19 pad 1: ROW1 -> Net-(D19-Pad1)
- D19 pad 2: Net-(D19-Pad2) -> ROW1
- D2 pad 1: ROW0 -> Net-(D2-Pad1)
- D2 pad 2: Net-(D2-Pad2) -> ROW0
- D20 pad 1: ROW1 -> Net-(D20-Pad1)
- D20 pad 2: Net-(D20-Pad2) -> ROW1
- D21 pad 1: ROW1 -> Net-(D21-Pad1)
- D21 pad 2: Net-(D21-Pad2) -> ROW1
- D22 pad 1: ROW1 -> Net-(D22-Pad1)
- D22 pad 2: Net-(D22-Pad2) -> ROW1
- D23 pad 1: ROW1 -> Net-(D23-Pad1)
- D23 pad 2: Net-(D23-Pad2) -> ROW1
- D24 pad 1: ROW1 -> Net-(D24-Pad1)
- D24 pad 2: Net-(D24-Pad2) -> ROW1
- D25 pad 1: ROW1 -> Net-(D25-Pad1)
- D25 pad 2: Net-(D25-Pad2) -> ROW1
- D26 pad 1: ROW1 -> Net-(D26-Pad1)
- D26 pad 2: Net-(D26-Pad2) -> ROW1
- D27 pad 1: ROW1 -> Net-(D27-Pad1)
- D27 pad 2: Net-(D27-Pad2) -> ROW1
- D28 pad 1: ROW1 -> Net-(D28-Pad1)
- D28 pad 2: Net-(D28-Pad2) -> ROW1
- D29 pad 1: ROW1 -> Net-(D29-Pad1)
- D29 pad 2: Net-(D29-Pad2) -> ROW1
- D3 pad 1: ROW0 -> Net-(D3-Pad1)
- D3 pad 2: Net-(D3-Pad2) -> ROW0
- D30 pad 1: ROW1 -> Net-(D30-Pad1)
- D30 pad 2: Net-(D30-Pad2) -> ROW1
- D31 pad 1: ROW2 -> Net-(D31-Pad1)
- D31 pad 2: Net-(D31-Pad2) -> ROW2
- D32 pad 1: ROW2 -> Net-(D32-Pad1)
- D32 pad 2: Net-(D32-Pad2) -> ROW2
- D33 pad 1: ROW2 -> Net-(D33-Pad1)
- D33 pad 2: Net-(D33-Pad2) -> ROW2
- D34 pad 1: ROW2 -> Net-(D34-Pad1)
- D34 pad 2: Net-(D34-Pad2) -> ROW2
- D35 pad 1: ROW2 -> Net-(D35-Pad1)
- D35 pad 2: Net-(D35-Pad2) -> ROW2
- D36 pad 1: ROW2 -> Net-(D36-Pad1)
- D36 pad 2: Net-(D36-Pad2) -> ROW2
- D37 pad 1: ROW2 -> Net-(D37-Pad1)
- D37 pad 2: Net-(D37-Pad2) -> ROW2
- D38 pad 1: ROW2 -> Net-(D38-Pad1)
- D38 pad 2: Net-(D38-Pad2) -> ROW2
- D39 pad 1: ROW2 -> Net-(D39-Pad1)
- D39 pad 2: Net-(D39-Pad2) -> ROW2
- D4 pad 1: ROW0 -> Net-(D4-Pad1)
- D4 pad 2: Net-(D4-Pad2) -> ROW0
- D40 pad 1: ROW2 -> Net-(D40-Pad1)
- D40 pad 2: Net-(D40-Pad2) -> ROW2
- D41 pad 1: ROW2 -> Net-(D41-Pad1)
- D41 pad 2: Net-(D41-Pad2) -> ROW2
- D42 pad 1: ROW2 -> Net-(D42-Pad1)
- D42 pad 2: Net-(D42-Pad2) -> ROW2
- D43 pad 1: ROW2 -> Net-(D43-Pad1)
- D43 pad 2: Net-(D43-Pad2) -> ROW2
- D44 pad 1: ROW2 -> Net-(D44-Pad1)
- D44 pad 2: Net-(D44-Pad2) -> ROW2
- D45 pad 1: ROW2 -> Net-(D45-Pad1)
- D45 pad 2: Net-(D45-Pad2) -> ROW2
- D46 pad 1: ROW3 -> Net-(D46-Pad1)
- D46 pad 2: Net-(D46-Pad2) -> ROW3
- D47 pad 1: ROW3 -> Net-(D47-Pad1)
- D47 pad 2: Net-(D47-Pad2) -> ROW3
- D48 pad 1: ROW3 -> Net-(D48-Pad1)
- D48 pad 2: Net-(D48-Pad2) -> ROW3
- D49 pad 1: ROW3 -> Net-(D49-Pad1)
- D49 pad 2: Net-(D49-Pad2) -> ROW3
- D5 pad 1: ROW0 -> Net-(D5-Pad1)
- D5 pad 2: Net-(D5-Pad2) -> ROW0
- D50 pad 1: ROW3 -> Net-(D50-Pad1)
- D50 pad 2: Net-(D50-Pad2) -> ROW3
- D51 pad 1: ROW3 -> Net-(D51-Pad1)
- D51 pad 2: Net-(D51-Pad2) -> ROW3
- D52 pad 1: ROW3 -> Net-(D52-Pad1)
- D52 pad 2: Net-(D52-Pad2) -> ROW3
- D53 pad 1: ROW3 -> Net-(D53-Pad1)
- D53 pad 2: Net-(D53-Pad2) -> ROW3
- D54 pad 1: ROW3 -> Net-(D54-Pad1)
- D54 pad 2: Net-(D54-Pad2) -> ROW3
- D55 pad 1: ROW3 -> Net-(D55-Pad1)
- D55 pad 2: Net-(D55-Pad2) -> ROW3
- D56 pad 1: ROW3 -> Net-(D56-Pad1)
- D56 pad 2: Net-(D56-Pad2) -> ROW3
- D57 pad 1: ROW3 -> Net-(D57-Pad1)
- D57 pad 2: Net-(D57-Pad2) -> ROW3
- D58 pad 1: ROW3 -> Net-(D58-Pad1)
- D58 pad 2: Net-(D58-Pad2) -> ROW3
- D59 pad 1: ROW3 -> Net-(D59-Pad1)
- D59 pad 2: Net-(D59-Pad2) -> ROW3
- D6 pad 1: ROW0 -> Net-(D6-Pad1)
- D6 pad 2: Net-(D6-Pad2) -> ROW0
- D60 pad 1: ROW3 -> Net-(D60-Pad1)
- D60 pad 2: Net-(D60-Pad2) -> ROW3
- D61 pad 1: ROW4 -> Net-(D61-Pad1)
- D61 pad 2: Net-(D61-Pad2) -> ROW4
- D62 pad 1: ROW4 -> Net-(D62-Pad1)
- D62 pad 2: Net-(D62-Pad2) -> ROW4
- D63 pad 1: ROW4 -> Net-(D63-Pad1)
- D63 pad 2: Net-(D63-Pad2) -> ROW4
- D64 pad 1: ROW4 -> Net-(D64-Pad1)
- D64 pad 2: Net-(D64-Pad2) -> ROW4
- D65 pad 1: ROW4 -> Net-(D65-Pad1)
- D65 pad 2: Net-(D65-Pad2) -> ROW4
- D66 pad 1: ROW4 -> Net-(D66-Pad1)
- D66 pad 2: Net-(D66-Pad2) -> ROW4
- D67 pad 1: ROW4 -> Net-(D67-Pad1)
- D67 pad 2: Net-(D67-Pad2) -> ROW4
- D68 pad 1: ROW4 -> Net-(D68-Pad1)
- D68 pad 2: Net-(D68-Pad2) -> ROW4
- D69 pad 1: ROW4 -> Net-(D69-Pad1)
- D69 pad 2: Net-(D69-Pad2) -> ROW4
- D7 pad 1: ROW0 -> Net-(D7-Pad1)
- D7 pad 2: Net-(D7-Pad2) -> ROW0
- D70 pad 1: ROW4 -> Net-(D70-Pad1)
- D70 pad 2: Net-(D70-Pad2) -> ROW4
- D71 pad 1: ROW4 -> Net-(D71-Pad1)
- D71 pad 2: Net-(D71-Pad2) -> ROW4
- D72 pad 1: ROW4 -> Net-(D72-Pad1)
- D72 pad 2: Net-(D72-Pad2) -> ROW4
- D73 pad 1: ROW4 -> Net-(D73-Pad1)
- D73 pad 2: Net-(D73-Pad2) -> ROW4
- D74 pad 1: ROW4 -> Net-(D74-Pad1)
- D74 pad 2: Net-(D74-Pad2) -> ROW4
- D75 pad 1: ROW4 -> Net-(D75-Pad1)
- D75 pad 2: Net-(D75-Pad2) -> ROW4
- D8 pad 1: ROW0 -> Net-(D8-Pad1)
- D8 pad 2: Net-(D8-Pad2) -> ROW0
- D9 pad 1: ROW0 -> Net-(D9-Pad1)
- D9 pad 2: Net-(D9-Pad2) -> ROW0
- SW10 pad 1: Net-(D9-Pad2) -> Net-(D9-Pad1)
- SW11 pad 1: Net-(D10-Pad2) -> Net-(D10-Pad1)
- SW12 pad 1: Net-(D11-Pad2) -> Net-(D11-Pad1)
- SW13 pad 1: Net-(D12-Pad2) -> Net-(D12-Pad1)
- SW14 pad 1: Net-(D13-Pad2) -> Net-(D13-Pad1)
- SW16 pad 1: Net-(D15-Pad2) -> Net-(D15-Pad1)
- SW17 pad 1: Net-(D16-Pad2) -> Net-(D16-Pad1)
- SW18 pad 1: Net-(D17-Pad2) -> Net-(D17-Pad1)
- SW19 pad 1: Net-(D18-Pad2) -> Net-(D18-Pad1)
- SW2 pad 1: Net-(D1-Pad2) -> Net-(D1-Pad1)
- SW20 pad 1: Net-(D19-Pad2) -> Net-(D19-Pad1)
- SW21 pad 1: Net-(D20-Pad2) -> Net-(D20-Pad1)
- SW22 pad 1: Net-(D21-Pad2) -> Net-(D21-Pad1)
- SW23 pad 1: Net-(D22-Pad2) -> Net-(D22-Pad1)
- SW24 pad 1: Net-(D23-Pad2) -> Net-(D23-Pad1)
- SW25 pad 1: Net-(D24-Pad2) -> Net-(D24-Pad1)
- SW26 pad 1: Net-(D25-Pad2) -> Net-(D25-Pad1)
- SW27 pad 1: Net-(D26-Pad2) -> Net-(D26-Pad1)
- SW28 pad 1: Net-(D27-Pad2) -> Net-(D27-Pad1)
- SW29 pad 1: Net-(D28-Pad2) -> Net-(D28-Pad1)
- SW3 pad 1: Net-(D2-Pad2) -> Net-(D2-Pad1)
- SW30 pad 1: Net-(D29-Pad2) -> Net-(D29-Pad1)
- SW31 pad 1: Net-(D30-Pad2) -> Net-(D30-Pad1)
- SW32 pad 1: Net-(D31-Pad2) -> Net-(D31-Pad1)
- SW33 pad 1: Net-(D32-Pad2) -> Net-(D32-Pad1)
- SW34 pad 1: Net-(D33-Pad2) -> Net-(D33-Pad1)
- SW35 pad 1: Net-(D34-Pad2) -> Net-(D34-Pad1)
- SW36 pad 1: Net-(D35-Pad2) -> Net-(D35-Pad1)
- SW37 pad 1: Net-(D36-Pad2) -> Net-(D36-Pad1)
- SW38 pad 1: Net-(D37-Pad2) -> Net-(D37-Pad1)
- SW39 pad 1: Net-(D38-Pad2) -> Net-(D38-Pad1)
- SW4 pad 1: Net-(D3-Pad2) -> Net-(D3-Pad1)
- SW40 pad 1: Net-(D39-Pad2) -> Net-(D39-Pad1)
- SW41 pad 1: Net-(D40-Pad2) -> Net-(D40-Pad1)
- SW42 pad 1: Net-(D41-Pad2) -> Net-(D41-Pad1)
- SW43 pad 1: Net-(D42-Pad2) -> Net-(D42-Pad1)
- SW44 pad 1: Net-(D43-Pad2) -> Net-(D43-Pad1)
- SW45 pad 1: Net-(D44-Pad2) -> Net-(D44-Pad1)
- SW46 pad 1: Net-(D45-Pad2) -> Net-(D45-Pad1)
- SW47 pad 1: Net-(D46-Pad2) -> Net-(D46-Pad1)
- SW48 pad 1: Net-(D47-Pad2) -> Net-(D47-Pad1)
- SW49 pad 1: Net-(D48-Pad2) -> Net-(D48-Pad1)
- SW5 pad 1: Net-(D4-Pad2) -> Net-(D4-Pad1)
- SW50 pad 1: Net-(D49-Pad2) -> Net-(D49-Pad1)
- SW51 pad 1: Net-(D50-Pad2) -> Net-(D50-Pad1)
- SW52 pad 1: Net-(D51-Pad2) -> Net-(D51-Pad1)
- SW53 pad 1: Net-(D52-Pad2) -> Net-(D52-Pad1)
- SW54 pad 1: Net-(D53-Pad2) -> Net-(D53-Pad1)
- SW55 pad 1: Net-(D54-Pad2) -> Net-(D54-Pad1)
- SW56 pad 1: Net-(D55-Pad2) -> Net-(D55-Pad1)
- SW57 pad 1: Net-(D56-Pad2) -> Net-(D56-Pad1)
- SW58 pad 1: Net-(D57-Pad2) -> Net-(D57-Pad1)
- SW59 pad 1: Net-(D58-Pad2) -> Net-(D58-Pad1)
- SW6 pad 1: Net-(D5-Pad2) -> Net-(D5-Pad1)
- SW60 pad 1: Net-(D59-Pad2) -> Net-(D59-Pad1)
- SW61 pad 1: Net-(D60-Pad2) -> Net-(D60-Pad1)
- SW62 pad 1: Net-(D61-Pad2) -> Net-(D61-Pad1)
- SW63 pad 1: Net-(D62-Pad2) -> Net-(D62-Pad1)
- SW64 pad 1: Net-(D63-Pad2) -> Net-(D63-Pad1)
- SW65 pad 1: Net-(D64-Pad2) -> Net-(D64-Pad1)
- SW66 pad 1: Net-(D65-Pad2) -> Net-(D65-Pad1)
- SW67 pad 1: Net-(D66-Pad2) -> Net-(D66-Pad1)
- SW68 pad 1: Net-(D67-Pad2) -> Net-(D67-Pad1)
- SW69 pad 1: Net-(D68-Pad2) -> Net-(D68-Pad1)
- SW7 pad 1: Net-(D6-Pad2) -> Net-(D6-Pad1)
- SW70 pad 1: Net-(D69-Pad2) -> Net-(D69-Pad1)
- SW71 pad 1: Net-(D70-Pad2) -> Net-(D70-Pad1)
- SW72 pad 1: Net-(D71-Pad2) -> Net-(D71-Pad1)
- SW73 pad 1: Net-(D72-Pad2) -> Net-(D72-Pad1)
- SW74 pad 1: Net-(D73-Pad2) -> Net-(D73-Pad1)
- SW75 pad 1: Net-(D74-Pad2) -> Net-(D74-Pad1)
- SW76 pad 1: Net-(D75-Pad2) -> Net-(D75-Pad1)
- SW8 pad 1: Net-(D7-Pad2) -> Net-(D7-Pad1)
- SW9 pad 1: Net-(D8-Pad2) -> Net-(D8-Pad1)
Routing:
- net aCS5: track 228.9 -> 208.3 mm
- net aCS10: track 152.5 -> 143.8 mm, vias 10 -> 7
- net Net-(D71-Pad2): track 6.83 -> 0.00 mm
- net Net-(D23-Pad2): track 6.42 -> 0.00 mm
- net Net-(D33-Pad2): track 6.26 -> 0.00 mm
- net Net-(D33-Pad1): track 0.00 -> 6.16 mm
- net Net-(D1-Pad2): track 5.95 -> 0.00 mm
- net Net-(D71-Pad1): track 0.00 -> 5.83 mm
- net aSW4: track 364.7 -> 370.4 mm
- net Net-(D1-Pad1): track 0.00 -> 5.63 mm
- net Net-(D46-Pad1): track 0.00 -> 5.57 mm
- net Net-(D23-Pad1): track 0.00 -> 5.52 mm
- net Net-(D7-Pad2): track 5.50 -> 0.00 mm
- net Net-(D10-Pad2): track 5.50 -> 0.00 mm
- net bCS5: track 155.0 -> 149.5 mm
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
Commit message: Delete old gerbers
Routing:
- net bCS5: track 149.5 -> 151.0 mm, vias 7 -> 9
- net aCS10: track 143.8 -> 145.0 mm
- net GND: vias 442 -> 440
- removed copper zone on F.Cu, net GND
Other:
- net class Default: clearance 0.2 -> 0.15
- net class Power: clearance 0.2 -> 0.15
- rule trace_clearance: 0.2 -> 0.15
