File: qs75.kicad_pcb (KiCad board)
At the start: 2 copper layers, 285 x 95.1 mm, 284 parts, among them J1 SWD, J2 SPI, J3 UART, J4 USB2.0, J5 PB14, SW1 SW_Push, SW10 1u, SW11 1u, SW12 1u, SW13 1u, SW14 1u, SW15 1u, SW16 1u, SW17 1u, SW18 1u, SW19 1u, SW2 1u, SW20 1u, SW21 1u, SW22 1u, SW23 1u, SW24 1u, SW25 1u, SW26 1u, SW27 1u, SW28 1u, SW29 1u, SW3 1u, SW30 1u, SW31 1u, SW32 1u, SW33 1u, SW34 1u, SW35 1u, SW36 1u, SW37 1u, SW38 1u, SW39 1u, SW4 1u, SW40 1u, SW41 1u, SW42 1u, SW43 1u, SW44 1u, SW45 1u, SW46 1u, SW47 1u, SW48 1u, SW49 1u, SW5 1u, SW50 1u, SW51 1u, SW52 1u, SW53 1u, SW54 1u, SW55 1u, SW56 1u, SW57 1u, SW58 1u, SW59 1u, SW6 1u, SW60 1u, SW61 1u, SW62 1u, SW63 1u, SW64 1u, SW65 1u, SW66 1u, SW67 1u, SW68 1u, SW69 1u, SW7 1u, SW70 1u, SW71 1u, SW72 1u, SW73 1u, SW74 1u, SW75 1u, SW76 1u, SW77 SW_Push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

Commit message: Add holes for GH60-case
Parts:
- added HOLE: VAL**, hole:PKRH, F.Cu at (266.8, 47.8)
- added HOLE: VAL**, hole:PKRHC, F.Cu at (31.9, 47.8)
- added HOLE: VAL**, hole:PKRH, F.Cu at (134.9, 66.9)
Routing:
- net aSW4: track 370.4 -> 437.9 mm
- net aSW8: track 395.9 -> 401.6 mm
- net bSW6: track 288.4 -> 294.0 mm
- net aSW5: track 348.5 -> 353.4 mm, vias 8 -> 10
- net +3V3: track 662.4 -> 658.0 mm
- net SCK: track 39.0 -> 41.4 mm
- net ROW1: track 415.6 -> 417.8 mm
- net NSS: track 46.4 -> 48.2 mm
- net aSW7: track 424.7 -> 426.2 mm, vias 20 -> 18
- net aCS2: track 143.8 -> 144.6 mm
- net ROW2: track 358.0 -> 358.7 mm
- net GND: vias 441 -> 445
